File: schematic/ESP8266 Wiring.sch (EAGLE design)
At the start: 9 parts

Commit message: Prototype release
Other:
- note added: "http://resterampeberlin.wordpress.com"
Changed lines of the file:
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@@
 <part name="GND1" library="supply1" deviceset="GND" device=""/>
 <part name="POWER" library="con-lstb" deviceset="MA03-1" device=""/>
+<part name="FRAME1" library="frames" deviceset="DINA4_L" device=""/>
 </parts>
 <sheets>
@@
 <text x="-25.4" y="83.82" size="1.778" layer="96">RX</text>
 <text x="-25.4" y="81.28" size="1.778" layer="97">TX</text>
+<text x="83.82" y="10.16" size="3.81" layer="97">http://resterampeberlin.wordpress.com</text>
 </plain>
 <instances>
@@
 <instance part="GND1" gate="1" x="40.64" y="55.88"/>
 <instance part="POWER" gate="G$1" x="-20.32" y="101.6"/>
+<instance part="FRAME1" gate="G$1" x="-81.28" y="-15.24"/>
+<instance part="FRAME1" gate="G$2" x="81.28" y="-15.24"/>
 </instances>
 <busses>
