File: schematic/Roomsensor.sch (EAGLE design)
At the start: 16 parts

Commit message: Prototype release
Parts:
- removed LED1: (no value), led:LED3MM
- R4: value 270 -> 4,7K
Connections:
- removed net N$1: LED1.A, R4.1
- removed net N$2: R4.2, U$1.GPIO2
- net 1WIRE: now also R4.1, U$1.GPIO2
- net GND: no longer LED1.C
- net VCC: now also R4.2
Other:
- note added: "http://resterampeberlin.wordpress.com"
- moved on the sheet: R4
Changed lines of the file:
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@@
 <part name="GND1" library="supply1" deviceset="GND" device=""/>
 <part name="POWER" library="con-lstb" deviceset="MA03-1" device=""/>
-<part name="LED1" library="led" deviceset="LED" device="3MM"/>
-<part name="R4" library="resistor" deviceset="R-EU_" device="0207/10" value="270"/>
 <part name="U1" library="merriman" deviceset="18S20" device=""/>
 <part name="U2" library="merriman" deviceset="18S20" device=""/>
@@
 <part name="P+2" library="supply1" deviceset="VCC" device="" value="3,3V"/>
 <part name="GND2" library="supply1" deviceset="GND" device=""/>
+<part name="R4" library="resistor" deviceset="R-EU_" device="0207/10" value="4,7K"/>
+<part name="FRAME1" library="frames" deviceset="DINA4_L" device=""/>
 </parts>
 <sheets>
@@
 <text x="-25.4" y="83.82" size="1.778" layer="96">RX</text>
 <text x="-25.4" y="81.28" size="1.778" layer="97">TX</text>
+<text x="71.12" y="-15.24" size="3.81" layer="97" distance="85">http://resterampeberlin.wordpress.com</text>
 </plain>
 <instances>
@@
 <instance part="GND1" gate="1" x="40.64" y="50.8"/>
 <instance part="POWER" gate="G$1" x="-20.32" y="101.6"/>
-<instance part="LED1" gate="G$1" x="27.94" y="66.04"/>
-<instance part="R4" gate="G$1" x="27.94" y="73.66" rot="R90"/>
 <instance part="U1" gate="18S20" x="-17.78" y="22.86"/>
 <instance part="U2" gate="18S20" x="12.7" y="22.86"/>
@@
 <instance part="P+2" gate="VCC" x="40.64" y="43.18"/>
 <instance part="GND2" gate="1" x="40.64" y="-2.54"/>
+<instance part="R4" gate="G$1" x="-38.1" y="25.4" rot="R90"/>
+<instance part="FRAME1" gate="G$1" x="-93.98" y="-43.18"/>
+<instance part="FRAME1" gate="G$2" x="68.58" y="-43.18"/>
 </instances>
 <busses>
@@
 <wire x1="40.64" y1="35.56" x2="68.58" y2="35.56" width="0.1524" layer="91"/>
 <junction x="68.58" y="35.56"/>
+<wire x1="-17.78" y1="35.56" x2="-38.1" y2="35.56" width="0.1524" layer="91"/>
+<junction x="-17.78" y="35.56"/>
+<pinref part="R4" gate="G$1" pin="2"/>
+<wire x1="-38.1" y1="35.56" x2="-38.1" y2="30.48" width="0.1524" layer="91"/>
 </segment>
 </net>
@@
 <wire x1="15.24" y1="58.42" x2="22.86" y2="58.42" width="0.1524" layer="91"/>
 <pinref part="U$1" gate="G$1" pin="GND"/>
-<wire x1="22.86" y1="58.42" x2="27.94" y2="58.42" width="0.1524" layer="91"/>
-<wire x1="27.94" y1="58.42" x2="40.64" y2="58.42" width="0.1524" layer="91"/>
+<wire x1="22.86" y1="58.42" x2="40.64" y2="58.42" width="0.1524" layer="91"/>
 <wire x1="40.64" y1="58.42" x2="68.58" y2="58.42" width="0.1524" layer="91"/>
 <wire x1="30.48" y1="88.9" x2="22.86" y2="88.9" width="0.1524" layer="91"/>
@@
 <wire x1="-7.62" y1="99.06" x2="-7.62" y2="78.74" width="0.1524" layer="91"/>
 <junction x="-7.62" y="78.74"/>
-<pinref part="LED1" gate="G$1" pin="C"/>
-<wire x1="27.94" y1="60.96" x2="27.94" y2="58.42" width="0.1524" layer="91"/>
-<junction x="27.94" y="58.42"/>
 </segment>
 <segment>
@@
 </segment>
 </net>
-<net name="N$1" class="0">
-<segment>
-<pinref part="LED1" gate="G$1" pin="A"/>
-<pinref part="R4" gate="G$1" pin="1"/>
-</segment>
-</net>
-<net name="N$2" class="0">
-<segment>
-<pinref part="U$1" gate="G$1" pin="GPIO2"/>
-<wire x1="30.48" y1="86.36" x2="27.94" y2="86.36" width="0.1524" layer="91"/>
-<pinref part="R4" gate="G$1" pin="2"/>
-<wire x1="27.94" y1="86.36" x2="27.94" y2="78.74" width="0.1524" layer="91"/>
-</segment>
-</net>
 <net name="1WIRE" class="0">
 <segment>
 <pinref part="U1" gate="18S20" pin="DQ"/>
 <wire x1="-30.48" y1="22.86" x2="-30.48" y2="5.08" width="0.1524" layer="91"/>
-<wire x1="-30.48" y1="5.08" x2="-40.64" y2="5.08" width="0.1524" layer="91"/>
+<wire x1="-30.48" y1="5.08" x2="-38.1" y2="5.08" width="0.1524" layer="91"/>
 <junction x="-30.48" y="5.08"/>
-<label x="-40.64" y="5.08" size="1.778" layer="95"/>
+<label x="-50.8" y="5.08" size="1.778" layer="95"/>
+<wire x1="-38.1" y1="5.08" x2="-50.8" y2="5.08" width="0.1524" layer="91"/>
 <wire x1="25.4" y1="5.08" x2="-2.54" y2="5.08" width="0.1524" layer="91"/>
 <wire x1="-2.54" y1="5.08" x2="-30.48" y2="5.08" width="0.1524" layer="91"/>
@@
 <wire x1="-2.54" y1="22.86" x2="-2.54" y2="5.08" width="0.1524" layer="91"/>
 <junction x="-2.54" y="5.08"/>
-</segment>
-</net>
+<pinref part="R4" gate="G$1" pin="1"/>
+<wire x1="-38.1" y1="20.32" x2="-38.1" y2="5.08" width="0.1524" layer="91"/>
+<junction x="-38.1" y="5.08"/>
+</segment>
+<segment>
+<pinref part="U$1" gate="G$1" pin="GPIO2"/>
+<wire x1="30.48" y1="86.36" x2="25.4" y2="86.36" width="0.1524" layer="91"/>
+<wire x1="25.4" y1="86.36" x2="25.4" y2="53.34" width="0.1524" layer="91"/>
+<wire x1="25.4" y1="53.34" x2="-7.62" y2="53.34" width="0.1524" layer="91"/>
+<label x="-7.62" y="53.34" size="1.778" layer="95"/>
+</segment>
+</net>
